File: hcde598/hw05/wing/wing.kicad_pcb (KiCad board)
At the start: 2 copper layers, 28 x 5.3 mm, 0 parts

Commit message: Pivot back to mac, grab some pics
Other:
- board size 28 x 5.3 mm -> 59.8 x 6.2 mm
