File: hcde598/hw08/horizontal-stabilizer/horizontal-stabilizer.kicad_pcb (KiCad board)
At the start: 2 copper layers, 72.3 x 32.8 mm, 0 parts

Commit message: Last commit for Monday
Other:
- board size 72.3 x 32.8 mm -> 37.4 x 12.2 mm
